File: hardware/PurplePaddock/5v_power.kicad_sch (KiCad schematic)
At the start: 0 parts

Commit message: Schematics, GPIO, Motor sensing, LED sensing, status LEDs and PWM
Parts:
- added C12: 470uF, symbol Device:C_Polarized
- added C13: 180uF, symbol Device:C_Polarized
- added C14: 180uF, symbol Device:C
- added C15: 2.2uF, symbol Device:C
- added D5: D_Schottky, symbol Device:D_Schottky
- added L3: 220uH, symbol Device:L
- added L4: 3uH, symbol Device:L
- added R27: 5.0k, symbol Device:R
- added R28: 1.2k, symbol Device:R
- added U2: LM2596S-ADJ, Package_TO_SOT_SMD:TO-263-5_TabPin3, symbol Regulator_Switching:LM2596S-ADJ
Connections:
- new net: D5.1 (K), L3.1, U2.2 (OUT)
- new net GND: C12.2, C13.2, C14.2, D5.2 (A), R28.2, U2.3 (GND), U2.5 (~{ON}/OFF)
- new net MOCK_BATT_OUT: C14.1, L4.2
- new net PWR_IN: C12.1, U2.1 (VIN)
- new net buck_out: C13.1, C15.1, L3.2, L4.1, R27.1
- new net feedback: C15.2, R27.2, R28.1, U2.4 (FB)
Other:
- note added: "A 1st order low pass filter, value suggested from LM2596 datasheet. Values not too important, capacitor should be very low ESR."
- note added: "Buck Converter"
- note added: "Feedback"
- note added: "Feedback ensures buck out is 5.1V."
- note added: "Needs a ripple current rating of >50% of the DC current rating"
- note added: "Output filter"
- note added: "TODO recalculate all of these values for 5V"
- note added: "Want a closed core magnetic inductor"
