File: hardware/PurplePaddock/PurplePaddock.kicad_sch (KiCad schematic)
At the start: 5 parts, among them P1 Conn_02x20_Odd_Even

Commit message: Schematics, GPIO, Motor sensing, LED sensing, status LEDs and PWM
Parts:
- added D2: LED_Dual_AAK, symbol Device:LED_Dual_AAK
- added D3, D4: LED, symbol Device:LED
- added J1, J2, J3, J5: Conn_01x03_Male, symbol Connector:Conn_01x03_Male
- added J10: Barrel_Jack, symbol Connector:Barrel_Jack
- added J4, J8, J9: Conn_01x02_Female, symbol Connector:Conn_01x02_Female
- added J7: Conn_01x02, symbol Connector_Generic:Conn_01x02
- added R10, R11, R12, R13: R, symbol Device:R
- added R14, R15, R16, R17: R_Photo, symbol Device:R_Photo
- added R18: 10k, symbol Device:R
- added R19: 2.2k, symbol Device:R
- added R24, R25, R26: 150, symbol Device:R
Connections:
- net +5V: now also R10.1, R11.1, R12.1, R13.1, R24.1
- net GND: now also D3.1 (K), D4.1 (K), J10.2, J7.2 (Pin_2), R14.2, R15.2, R16.2, R17.2, R19.1, R26.2
- net battery_simulator/MOCK_BATT_OUT: now also J7.1 (Pin_1)
- new net: D2.3 (K), R26.1
- new net: D4.2 (A), R25.2
- new net: D3.2 (A), R24.2
- new net FAIL: D2.1 (A1)
- new net PASS: D2.2 (A2)
- new net PWR_IN: J10.1
- new net Power Button/SIDE_A: J9.2 (Pin_2)
- new net Power Button/SIDE_B: J9.1 (Pin_1)
- new net STATUS: R25.1
- new net SUT_12V: J4.2 (Pin_2), R18.2
- new net SUT_12V_Divided: R18.1, R19.2
- new net SUT_12V_GND: J4.1 (Pin_1)
- new net SUT_SERVO_1_5V: J1.1 (Pin_1)
- new net SUT_SERVO_1_GND: J1.3 (Pin_3)
- new net SUT_SERVO_1_PWM: J1.2 (Pin_2)
- new net SUT_SERVO_2_5V: J2.1 (Pin_1)
- new net SUT_SERVO_2_GND: J2.3 (Pin_3)
- new net SUT_SERVO_2_PWM: J2.2 (Pin_2)
- new net SUT_SERVO_3_5V: J3.1 (Pin_1)
- new net SUT_SERVO_3_GND: J3.3 (Pin_3)
- new net SUT_SERVO_3_PWM: J3.2 (Pin_2)
- new net SUT_SERVO_4_5V: J5.1 (Pin_1)
- new net SUT_SERVO_4_GND: J5.3 (Pin_3)
- new net SUT_SERVO_4_PWM: J5.2 (Pin_2)
- new net SUT_Status1_LED: R10.2, R14.1
- new net SUT_Status2_LED: R11.2, R15.1
- new net SUT_Status3_LED: R12.2, R16.1
- new net SUT_Status4_LED: R13.2, R17.1
- new net Start Button/SIDE_A: J8.2 (Pin_2)
- new net Start Button/SIDE_B: J8.1 (Pin_1)
Other:
- added sheet GPIO (gpio.kicad_sch)
- added sheet Motors1 (motors_1.kicad_sch)
- added sheet Motors2 (motors_1.kicad_sch)
- added sheet Power Button (mock_button.kicad_sch)
- added sheet Start Button (mock_button.kicad_sch)
- sheet 5v_power ports: added 5V, PWR_IN; removed none
- note added: "12V"
- note added: "Analogue comparitors can be used to ensure that the servo voltage rail and gnd have been soldered. This test is kind of null because I think that 4 servo motors should be connected anyway to check a brain was assembled right. We do not want to share a ground with the SUT other than the one provided in the powersupply inorder to prevent ground loops."
- note added: "Big PASS/FAIL LED"
- note added: "GPIO/BUTTONS"
- note added: "LEDS"
- note added: "POWER"
- note added: "RPi4B"
- note added: "RPi4B only Pi which can emulate a USB mass storage device and has 2 NIC's"
- note added: "SERVOS"
- note added: "SUT STATUS LED SENSING"
- note added: "The LDR's output is highly wavelength dependent. Changes in colour should corospond to changes in intensity Would take up alot of ADC inputs to do this though"
- note added: "The largest E12 ratio which ensures <3.3V out"
- note removed: "ID_SD and ID_SC PINS: These pins are reserved for HAT ID EEPROM. At boot time this I2C interface will be interrogated to look for an EEPROM that identifes the attached board and allows automagic setup of the GPIOs (and optionally, Linux drivers). DO NOT USE these pins for anything other than attaching an I2C ID EEPROM. Leave unconnected if ID EEPROM not required."
- moved on the sheet: MK1, MK2, MK3, MK4, P1
