File: hardware/Simulation/Battery_sim/battery_simulator.kicad_sch (KiCad schematic)
At the start: 14 parts, among them U1 LM2596S-ADJ

Commit message: Schematics, GPIO, Motor sensing, LED sensing, status LEDs and PWM
Parts:
- removed D1: D_Schottky, symbol Device:D_Schottky
- added D?: DIODE, symbol pspice:DIODE
- added V1: VDC, symbol Simulation_SPICE:VDC
- added V2: VPULSE, symbol Simulation_SPICE:VPULSE
- U1: Spice_Lib_File (none) -> C:\Users\edwin\Documents\libarries\LTSpice\LM2596_5P0_TRANS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; Spice_Model (none) -> LM2596_ADJ_TRANS; Spice_Netlist_Enabled (none) -> Y; Spice_Primitive (none) -> X
- gave numbers to parts that had none: 2
Connections:
- net GND: now also D?.1 (K), V1.2, V2.2
- net PWM_V_Ctrl: now also V2.1
- net PWR_IN: now also V1.1
- net at L1.1, U1.2 (OUT): now also D?.2 (A)
Other:
- note added: "SPICE"
- note removed: "Needs a ripple current rating of >50% of the DC current rating"
- note removed: "Want a closed core magnetic inductor"
